Commit message: Add controllers for Robotiq gripper palm joints

File: src/cobotics_control/urdf/rbkairos_kuka_iiwa_robotiq/rbkairos_kuka_iiwa_robotiq.xacro (robot description, xacro)
@@ -566,4 +566,15 @@
         </actuator>
     </transmission>
+    <!--<transmission name="palm_finger_middle_tran">
+        <robotNamespace>/iiwa</robotNamespace>
+        <type>transmission_interface/SimpleTransmission</type>
+        <joint name="palm_finger_middle_joint">
+            <hardwareInterface>EffortJointInterface</hardwareInterface>
+        </joint>
+        <actuator name="palm_finger_middle_motor">
+            <hardwareInterface>EffortJointInterface</hardwareInterface>
+            <mechanicalReduction>1</mechanicalReduction>
+        </actuator>
+    </transmission>-->
     <transmission name="finger_1_tran_1">
         <robotNamespace>/iiwa</robotNamespace>
