Commit message: Adding the orbbec astra camera topic in gazebo

File: src/robotnik/robotnik_sensors/urdf/orbbec_astra.urdf.xacro (robot description, xacro)
@@ -74,7 +74,7 @@
     </link>
   <!-- RGBD sensor for simulation, same as Kinect -->
-  <sensor_orbbec_astra_gazebo/>
+  <xacro:sensor_orbbec_astra_gazebo prefix="${prefix}" prefix_topic="${prefix_topic}" />
   </xacro:macro>
-   <xacro:macro name="sensor_orbbec_astra_gazebo">
+   <xacro:macro name="sensor_orbbec_astra_gazebo" params="prefix prefix_topic">
     <gazebo reference="${prefix}_link">
       <sensor type="depth" name="${prefix}_depth_sensor">

Commit message: Solved the issue related to the laser topics and added more depth to the simulated camera sensor

File: src/robotnik/robotnik_sensors/urdf/orbbec_astra.urdf.xacro (robot description, xacro)
@@ -90,5 +90,5 @@
           <clip>
             <near>0.05</near>
-            <far>3.5</far>
+            <far>8.0</far>
           </clip>
         </camera>

File: src/robotnik/robotnik_sensors/urdf/sick_s300.urdf.xacro (robot description, xacro)
@@ -42,7 +42,7 @@
 	<link name="${prefix}_link" />
 	<!-- Sick sensor sensor for simulation -->
-	<sensor_sick_s300_gazebo />
+	<xacro:sensor_sick_s300_gazebo prefix="${prefix}" prefix_topic="${prefix_topic}" gpu="${gpu}" />
   </xacro:macro>
-  <xacro:macro name="sensor_sick_s300_gazebo">
+  <xacro:macro name="sensor_sick_s300_gazebo" params="prefix prefix_topic gpu">
     <gazebo reference="${prefix}_link">
 		<xacro:if value="${gpu}">
